Commit message: Initial setup with moveit setup assistant

File: arm_urdf/urdf/arm.urdf (robot description, URDF)
Before this commit: robot robotic_arm_6dof , 5 links, 4 joints
Links:
- link arm_gripper: geometry collision mesh filename=package://arm_urdf/urdf/collision/Gripper-Simplified.stl scale=0.001 0.001 0.001; visual mesh filename=package://arm_urdf/urdf/visualization/Gripper-Simplified.stl scale=0.001 0.001 0.001
- link arm_link_0: geometry collision mesh filename=package://arm_urdf/urdf/collision/Shoulder-Simplified.stl scale=0.001 0.001 0.001; visual mesh filename=package://arm_urdf/urdf/visualization/Shoulder-Simplified.s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 scale=0.001 0.001 0.001
- link arm_link_1: geometry collision mesh filename=package://arm_urdf/urdf/collision/Long_Arm-Simplified.stl scale=0.001 0.001 0.001; visual mesh filename=package://arm_urdf/urdf/visualization/Long_Arm-Simplified.s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 scale=0.001 0.001 0.001
- link arm_link_2: geometry collision mesh filename=package://arm_urdf/urdf/collision/Short_Arm-Simplified.stl scale=0.001 0.001 0.001; visual mesh filename=package://arm_urdf/urdf/visualization/Short_Arm-Simplified.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 scale=0.001 0.001 0.001
- link base_link: geometry collision mesh filename=package://arm_urdf/urdf/collision/Base-Simplified.stl scale=0.001 0.001 0.001; visual mesh filename=package://arm_urdf/urdf/visualization/Base-Simplified.stl scale=0.001 0.001 0.001
Joints:
- joint elbow_pitch_joint: origin xyz=0.05925 0 0.36646 rpy=0 0 0 -> xyz=0.00725 0 0.36646 rpy=0 0 3.141592653589793
- joint shoulder_joint: origin xyz=0 0.1407 0 rpy=0 0 3.14159 -> xyz=0 -0.1407 0 rpy=0 0 1.57079632679
- joint wrist_pitch_joint: axis 0 0 1 -> 1 0 0; origin xyz=0.05325 0 0.24944 rpy=0 0 0 -> xyz=0.05325 0 0.24944 rpy=0 0 3.141592653589793
